File: MDBT40/breakout_MDBT40.sch (EAGLE design)
At the start: 17 parts

Commit message: Add update
Parts:
- removed 32.768LHZ: FC-12M, crystal:FC-12M
- removed P0_18, P0_19: (no value), led:LEDCHIP-LED0603
- removed R2, R3: (no value), adafruit:R-US_R0603
- removed U$2: SMTU2450-TOP, GClue-Supply:SMTU2450-TOP
- added CY1: CRYSTALABS07, FaBo-Crystal:CRYSTALABS07
- added U$8: SMTU-TOP2032, FaBo-Supply:SMTU-TOP2032
- U$3: value BREAKOUT_BLE_NORDIC -> BLE-BREAKOUT-NORDIC; device gclue:BREAKOUT_BLE_NORDIC -> FaBo-Template:BLE-BREAKOUT-NORDIC
Connections:
- removed net N$1: P0_18.A, R2.2
- removed net N$2: P0_19.A, R3.2
- net +3V3: now also U$8.+; no longer U$2.+
- net GND: now also U$8.-; no longer P0_18.C, P0_19.C, U$2.-
- net N$7: now also CY1.P$2; no longer 32.768LHZ.2
- net N$8: now also CY1.P$1; no longer 32.768LHZ.1
- net P0_00: now also U$3.P0_00; no longer U$3.P0_0
- net P0_01: now also U$3.P0_01; no longer U$3.P0_1
- net P0_02: now also U$3.P0_02; no longer U$3.P0_2
- net P0_03: now also U$3.P0_03; no longer U$3.P0_3
- net P0_04: now also U$3.P0_04; no longer U$3.P0_4
- net P0_05: now also U$3.P0_05; no longer U$3.P0_5
- net P0_06: now also U$3.P0_06; no longer U$3.P0_6
- net P0_07: now also U$3.P0_07; no longer U$3.P0_7
- net P0_08: now also U$3.P0_08; no longer U$3.P0_8
- net P0_09: now also U$3.P0_09
- net P0_18: no longer R2.1
- net P0_19: now also U$3.P0_19; no longer R3.1
Other:
- moved on the sheet: C3
