File: CCDBUGGER-TC2050/converter.sch (EAGLE design)
At the start: 4 parts

Commit message: Update new meme.
Parts:
- removed SERIAL: (no value), FaBo-Template:FABO_BRICK_SERIAL-CONNECTOR_I
- added ..: (no value), FaBo-Template:FABO_BRICK_SERIAL-S04B-PASK-2
Connections:
- net 3V3: now also ...VCC; no longer SERIAL.VCC
- net GND: now also ...GND; no longer SERIAL.GND
- net RX: now also ...RX; no longer SERIAL.RX
- net TX: now also ...TX; no longer SERIAL.TX
Changed lines of the file:
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@@
 <part name="U$4" library="GClue-Debbuger" deviceset="TC-2050-SOCKET" device=""/>
 <part name="." library="con-lstb" deviceset="MA06-1" device=""/>
-<part name="SERIAL" library="FaBo-Template" deviceset="FABO_BRICK_SERIAL" device="-CONNECTOR_I"/>
 <part name="GND1" library="FaBo-etc" deviceset="GND" device=""/>
 <part name="GND2" library="FaBo-etc" deviceset="GND" device=""/>
@@
 <part name="SUPPLY2" library="FaBo-etc" deviceset="3V3" device=""/>
 <part name="SUPPLY3" library="FaBo-etc" deviceset="3V3" device=""/>
+<part name=".." library="FaBo-Template" deviceset="FABO_BRICK_SERIAL" device="-S04B-PASK-2"/>
 </parts>
 <sheets>
@@
 <instance part="U$4" gate="G$1" x="109.22" y="53.34"/>
 <instance part="." gate="1" x="127" y="76.2" rot="R180"/>
-<instance part="SERIAL" gate="G$1" x="63.5" y="76.2"/>
 <instance part="GND1" gate="GND" x="81.28" y="63.5"/>
 <instance part="GND2" gate="GND" x="101.6" y="81.28"/>
@@
 <instance part="SUPPLY2" gate="3V3" x="88.9" y="76.2"/>
 <instance part="SUPPLY3" gate="3V3" x="106.68" y="83.82"/>
+<instance part=".." gate="G$1" x="60.96" y="76.2"/>
 </instances>
 <busses>
@@
 </segment>
 <segment>
-<pinref part="SERIAL" gate="G$1" pin="GND"/>
-<wire x1="71.12" y1="68.58" x2="81.28" y2="68.58" width="0.1524" layer="91"/>
+<wire x1="68.58" y1="68.58" x2="81.28" y2="68.58" width="0.1524" layer="91"/>
 <wire x1="81.28" y1="68.58" x2="81.28" y2="63.5" width="0.1524" layer="91"/>
 <pinref part="GND1" gate="GND" pin="GND"/>
+<pinref part=".." gate="G$1" pin="GND"/>
 </segment>
 </net>
@@
 </segment>
 <segment>
-<pinref part="SERIAL" gate="G$1" pin="TX"/>
-<wire x1="71.12" y1="78.74" x2="81.28" y2="78.74" width="0.1524" layer="91"/>
+<wire x1="68.58" y1="78.74" x2="81.28" y2="78.74" width="0.1524" layer="91"/>
 <label x="81.28" y="78.74" size="1.778" layer="95"/>
+<pinref part=".." gate="G$1" pin="TX"/>
 </segment>
 </net>
@@
 </segment>
 <segment>
-<pinref part="SERIAL" gate="G$1" pin="RX"/>
-<wire x1="71.12" y1="83.82" x2="81.28" y2="83.82" width="0.1524" layer="91"/>
+<wire x1="68.58" y1="83.82" x2="81.28" y2="83.82" width="0.1524" layer="91"/>
 <label x="81.28" y="83.82" size="1.778" layer="95"/>
+<pinref part=".." gate="G$1" pin="RX"/>
 </segment>
 </net>
@@
 </segment>
 <segment>
-<pinref part="SERIAL" gate="G$1" pin="VCC"/>
-<wire x1="71.12" y1="73.66" x2="88.9" y2="73.66" width="0.1524" layer="91"/>
+<wire x1="68.58" y1="73.66" x2="88.9" y2="73.66" width="0.1524" layer="91"/>
 <pinref part="SUPPLY2" gate="3V3" pin="3V3"/>
 <wire x1="88.9" y1="73.66" x2="88.9" y2="76.2" width="0.1524" layer="91"/>
+<pinref part=".." gate="G$1" pin="VCC"/>
 </segment>
 <segment>
