File: HTS221/HTS221_breakout.sch (EAGLE design)
At the start: 2 parts

Commit message: Update new meme.
Parts:
- removed .: ADA4075, FaBo-Opamp:ADA4075
- removed U$3: 8PIN, FaBo-Breakout:8PIN
- added HTS112: (no value), FaBo-Mems:ST-HTS221
- added U$1: 6PIN, FaBo-Breakout:6PIN
Connections:
- removed net 1: ..-IN, U$3.1
- removed net 2: ..G1, U$3.2
- removed net 3: ..G2, U$3.3
- removed net 4: ..+IN, U$3.4
- removed net 5: ..-VS, U$3.5
- removed net 6: ..REF, U$3.6
- removed net 7: ..VOUT, U$3.7
- removed net 8: ..+VS, U$3.8
- new net CS: HTS112.CS, U$1.6
- new net DRDY: HTS112.DRDY, U$1.3
- new net GND: HTS112.GND, U$1.5
- new net SCL: HTS112.SCL, U$1.2
- new net SDA: HTS112.SDA, U$1.4
- new net VDD: HTS112.VDD, U$1.1
Other:
- note removed: "1.0.0"
Changed lines of the file:
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@@
 <layer number="49" name="Reference" color="7" fill="1" visible="no" active="no"/>
 <layer number="50" name="dxf" color="7" fill="1" visible="no" active="no"/>
-<layer number="51" name="tDocu" color="14" fill="1" visible="no" active="no"/>
+<layer number="51" name="tDocu" color="7" fill="1" visible="no" active="no"/>
 <layer number="52" name="bDocu" color="7" fill="1" visible="no" active="no"/>
 <layer number="53" name="tGND_GNDA" color="7" fill="9" visible="no" active="no"/>
@@
 <layer number="154" name="FabDoc2" color="2" fill="1" visible="no" active="no"/>
 <layer number="155" name="FabDoc3" color="7" fill="15" visible="no" active="no"/>
-<layer number="160" name="O_Dim" color="12" fill="11" visible="yes" active="yes"/>
 <layer number="199" name="Contour" color="7" fill="1" visible="yes" active="yes"/>
-<layer number="200" name="200bmp" color="1" fill="10" visible="yes" active="yes"/>
+<layer number="200" name="200bmp" color="1" fill="10" visible="no" active="yes"/>
 <layer number="201" name="201bmp" color="2" fill="1" visible="no" active="no"/>
 <layer number="202" name="202bmp" color="3" fill="1" visible="no" active="no"/>
@@
 </classes>
 <parts>
-<part name="U$1" library="GClue" deviceset="A4L-LOC" device=""/>
-<part name="U$3" library="FaBo-Breakout" deviceset="8PIN" device=""/>
-<part name="." library="FaBo-Opamp" deviceset="ADA4075" device=""/>
+<part name="U$1" library="FaBo-Breakout" deviceset="6PIN" device=""/>
+<part name="HTS112" library="FaBo-Mems" deviceset="ST-HTS221" device=""/>
 </parts>
 <sheets>
 <sheet>
 <plain>
-<text x="246.38" y="20.32" size="2.54" layer="94" align="bottom-center">1.0.0</text>
 </plain>
 <instances>
-<instance part="U$1" gate="G$1" x="0" y="0"/>
-<instance part="U$3" gate="G$1" x="76.2" y="106.68"/>
-<instance part="." gate="G$1" x="76.2" y="137.16"/>
+<instance part="U$1" gate="G$1" x="43.18" y="68.58"/>
+<instance part="HTS112" gate="HTS221" x="43.18" y="43.18"/>
 </instances>
 <busses>
 </busses>
 <nets>
-<net name="1" class="0">
+<net name="VDD" class="0">
 <segment>
-<wire x1="63.5" y1="139.7" x2="53.34" y2="139.7" width="0.1524" layer="91"/>
-<label x="53.34" y="139.7" size="1.778" layer="95"/>
-<pinref part="." gate="G$1" pin="-IN"/>
+<pinref part="HTS112" gate="HTS221" pin="VDD"/>
+<wire x1="27.94" y1="45.72" x2="20.32" y2="45.72" width="0.1524" layer="91"/>
+<label x="20.32" y="45.72" size="1.778" layer="95"/>
 </segment>
 <segment>
-<wire x1="63.5" y1="109.22" x2="53.34" y2="109.22" width="0.1524" layer="91"/>
-<label x="53.34" y="109.22" size="1.778" layer="95"/>
-<pinref part="U$3" gate="G$1" pin="1"/>
+<pinref part="U$1" gate="G$1" pin="1"/>
+<wire x1="30.48" y1="71.12" x2="22.86" y2="71.12" width="0.1524" layer="91"/>
+<label x="22.86" y="71.12" size="1.778" layer="95"/>
 </segment>
 </net>
-<net name="2" class="0">
+<net name="SCL" class="0">
 <segment>
-<wire x1="63.5" y1="137.16" x2="53.34" y2="137.16" width="0.1524" layer="91"/>
-<label x="53.34" y="137.16" size="1.778" layer="95"/>
-<pinref part="." gate="G$1" pin="G1"/>
+<pinref part="HTS112" gate="HTS221" pin="SCL"/>
+<wire x1="27.94" y1="40.64" x2="20.32" y2="40.64" width="0.1524" layer="91"/>
+<label x="20.32" y="40.64" size="1.778" layer="95"/>
 </segment>
 <segment>
-<wire x1="63.5" y1="106.68" x2="53.34" y2="106.68" width="0.1524" layer="91"/>
-<label x="53.34" y="106.68" size="1.778" layer="95"/>
-<pinref part="U$3" gate="G$1" pin="2"/>
+<pinref part="U$1" gate="G$1" pin="2"/>
+<wire x1="30.48" y1="68.58" x2="22.86" y2="68.58" width="0.1524" layer="91"/>
+<label x="22.86" y="68.58" size="1.778" layer="95"/>
 </segment>
 </net>
-<net name="3" class="0">
+<net name="GND" class="0">
 <segment>
-<wire x1="63.5" y1="134.62" x2="53.34" y2="134.62" width="0.1524" layer="91"/>
-<label x="53.34" y="134.62" size="1.778" layer="95"/>
-<pinref part="." gate="G$1" pin="G2"/>
+<pinref part="HTS112" gate="HTS221" pin="GND"/>
+<wire x1="58.42" y1="45.72" x2="66.04" y2="45.72" width="0.1524" layer="91"/>
+<label x="66.04" y="45.72" size="1.778" layer="95"/>
 </segment>
 <segment>
-<wire x1="63.5" y1="104.14" x2="53.34" y2="104.14" width="0.1524" layer="91"/>
-<label x="53.34" y="104.14" size="1.778" layer="95"/>
-<pinref part="U$3" gate="G$1" pin="3"/>
+<pinref part="U$1" gate="G$1" pin="5"/>
+<wire x1="55.88" y1="68.58" x2="63.5" y2="68.58" width="0.1524" layer="91"/>
+<label x="63.5" y="68.58" size="1.778" layer="95"/>
 </segment>
 </net>
-<net name="4" class="0">
+<net name="SDA" class="0">
 <segment>
-<wire x1="63.5" y1="132.08" x2="53.34" y2="132.08" width="0.1524" layer="91"/>
-<label x="53.34" y="132.08" size="1.778" layer="95"/>
-<pinref part="." gate="G$1" pin="+IN"/>
+<pinref part="HTS112" gate="HTS221" pin="SDA"/>
+<wire x1="58.42" y1="40.64" x2="66.04" y2="40.64" width="0.1524" layer="91"/>
+<label x="66.04" y="40.64" size="1.778" layer="95"/>
 </segment>
 <segment>
-<wire x1="63.5" y1="101.6" x2="53.34" y2="101.6" width="0.1524" layer="91"/>
-<label x="53.34" y="101.6" size="1.778" layer="95"/>
-<pinref part="U$3" gate="G$1" pin="4"/>
+<pinref part="U$1" gate="G$1" pin="4"/>
+<wire x1="55.88" y1="66.04" x2="63.5" y2="66.04" width="0.1524" layer="91"/>
+<label x="63.5" y="66.04" size="1.778" layer="95"/>
 </segment>
 </net>
-<net name="8" class="0">
+<net name="DRDY" class="0">
 <segment>
-<wire x1="88.9" y1="109.22" x2="101.6" y2="109.22" width="0.1524" layer="91"/>
-<label x="101.6" y="109.22" size="1.778" layer="95"/>
-<pinref part="U$3" gate="G$1" pin="8"/>
+<pinref part="HTS112" gate="HTS221" pin="DRDY"/>
+<wire x1="43.18" y1="30.48" x2="43.18" y2="25.4" width="0.1524" layer="91"/>
+<label x="43.18" y="25.4" size="1.778" layer="95"/>
 </segment>
 <segment>
-<wire x1="88.9" y1="139.7" x2="99.06" y2="139.7" width="0.1524" layer="91"/>
-<label x="99.06" y="139.7" size="1.778" layer="95"/>
-<pinref part="." gate="G$1" pin="+VS"/>
+<pinref part="U$1" gate="G$1" pin="3"/>
+<wire x1="30.48" y1="66.04" x2="22.86" y2="66.04" width="0.1524" layer="91"/>
+<label x="22.86" y="66.04" size="1.778" layer="95"/>
 </segment>
 </net>
-<net name="7" class="0">
+<net name="CS" class="0">
 <segment>
-<wire x1="88.9" y1="106.68" x2="101.6" y2="106.68" width="0.1524" layer="91"/>
-<label x="101.6" y="106.68" size="1.778" layer="95"/>
-<pinref part="U$3" gate="G$1" pin="7"/>
+<pinref part="HTS112" gate="HTS221" pin="CS"/>
+<wire x1="43.18" y1="55.88" x2="43.18" y2="60.96" width="0.1524" layer="91"/>
+<label x="43.18" y="60.96" size="1.778" layer="95"/>
 </segment>
 <segment>
-<wire x1="88.9" y1="137.16" x2="99.06" y2="137.16" width="0.1524" layer="91"/>
-<label x="99.06" y="137.16" size="1.778" layer="95"/>
-<pinref part="." gate="G$1" pin="VOUT"/>
+<pinref part="U$1" gate="G$1" pin="6"/>
+<wire x1="55.88" y1="71.12" x2="63.5" y2="71.12" width="0.1524" layer="91"/>
+<label x="63.5" y="71.12" size="1.778" layer="95"/>
 </segment>
 </net>
-<net name="6" class="0">
-<segment>
-<wire x1="88.9" y1="104.14" x2="101.6" y2="104.14" width="0.1524" layer="91"/>
-<label x="101.6" y="104.14" size="1.778" layer="95"/>
-<pinref part="U$3" gate="G$1" pin="6"/>
-</segment>
-<segment>
-<wire x1="88.9" y1="134.62" x2="99.06" y2="134.62" width="0.1524" layer="91"/>
-<label x="99.06" y="134.62" size="1.778" layer="95"/>
-<pinref part="." gate="G$1" pin="REF"/>
-</segment>
-</net>
-<net name="5" class="0">
-<segment>
-<wire x1="88.9" y1="101.6" x2="101.6" y2="101.6" width="0.1524" layer="91"/>
-<label x="101.6" y="101.6" size="1.778" layer="95"/>
-<pinref part="U$3" gate="G$1" pin="5"/>
-</segment>
-<segment>
-<wire x1="88.9" y1="132.08" x2="99.06" y2="132.08" width="0.1524" layer="91"/>
-<label x="99.06" y="132.08" size="1.778" layer="95"/>
-<pinref part="." gate="G$1" pin="-VS"/>
-</segment>
-</net>
