File: JLINKLITE-TC2030/converter.sch (EAGLE design)
At the start: 4 parts

Commit message: Update new meme.
Parts:
- removed SERIAL: (no value), FaBo-Template:FABO_BRICK_SERIAL-CONNECTOR_I
- added ..: (no value), FaBo-Template:FABO_BRICK_SERIAL-S04B-PASK-2
Connections:
- net 3.3V: now also ...VCC; no longer SERIAL.VCC
- net GND: now also ...GND; no longer SERIAL.GND
- net RX: now also ...RX; no longer SERIAL.RX
- net TX: now also ...TX; no longer SERIAL.TX
Changed lines of the file:
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@@
 <part name="GND3" library="SparkFun" deviceset="GND" device=""/>
 <part name="P+2" library="SparkFun" deviceset="3.3V" device=""/>
-<part name="SERIAL" library="FaBo-Template" deviceset="FABO_BRICK_SERIAL" device="-CONNECTOR_I"/>
 <part name="GND4" library="SparkFun" deviceset="GND" device=""/>
 <part name="P+4" library="SparkFun" deviceset="3.3V" device=""/>
+<part name=".." library="FaBo-Template" deviceset="FABO_BRICK_SERIAL" device="-S04B-PASK-2"/>
 </parts>
 <sheets>
@@
 <instance part="GND3" gate="1" x="101.6" y="93.98"/>
 <instance part="P+2" gate="G$1" x="106.68" y="104.14"/>
-<instance part="SERIAL" gate="G$1" x="73.66" y="101.6"/>
 <instance part="GND4" gate="1" x="88.9" y="86.36"/>
 <instance part="P+4" gate="G$1" x="96.52" y="104.14"/>
+<instance part=".." gate="G$1" x="73.66" y="101.6"/>
 </instances>
 <busses>
@@
 </segment>
 <segment>
-<pinref part="SERIAL" gate="G$1" pin="GND"/>
 <wire x1="81.28" y1="93.98" x2="88.9" y2="93.98" width="0.1524" layer="91"/>
 <wire x1="88.9" y1="93.98" x2="88.9" y2="88.9" width="0.1524" layer="91"/>
 <pinref part="GND4" gate="1" pin="GND"/>
+<pinref part=".." gate="G$1" pin="GND"/>
 </segment>
 </net>
@@
 </segment>
 <segment>
-<pinref part="SERIAL" gate="G$1" pin="VCC"/>
 <wire x1="81.28" y1="99.06" x2="96.52" y2="99.06" width="0.1524" layer="91"/>
 <wire x1="96.52" y1="99.06" x2="96.52" y2="104.14" width="0.1524" layer="91"/>
 <pinref part="P+4" gate="G$1" pin="3.3V"/>
+<pinref part=".." gate="G$1" pin="VCC"/>
 </segment>
 </net>
@@
 </segment>
 <segment>
-<pinref part="SERIAL" gate="G$1" pin="TX"/>
 <wire x1="81.28" y1="104.14" x2="88.9" y2="104.14" width="0.1524" layer="91"/>
 <label x="88.9" y="104.14" size="1.778" layer="95"/>
+<pinref part=".." gate="G$1" pin="TX"/>
 </segment>
 </net>
@@
 </segment>
 <segment>
-<pinref part="SERIAL" gate="G$1" pin="RX"/>
 <wire x1="81.28" y1="109.22" x2="88.9" y2="109.22" width="0.1524" layer="91"/>
 <label x="88.9" y="109.22" size="1.778" layer="95"/>
+<pinref part=".." gate="G$1" pin="RX"/>
 </segment>
 </net>
