File: LP2985/LP2985_3v3.sch (EAGLE design)
At the start: 2 parts

Commit message: Update new meme.
Parts:
- removed .: ADA4075, FaBo-Opamp:ADA4075
- removed U$3: 8PIN, FaBo-Breakout:8PIN
- added C3, C4: 1uf, GClue-Capacitor:CAPACITOR0603
- added U$2: 4PIN-REGULATOR, FaBo-Breakout:4PIN-REGULATOR
- added U1: (no value), FaBo-Supply:LP2985-33DBVR
Connections:
- removed net 1: ..-IN, U$3.1
- removed net 2: ..G1, U$3.2
- removed net 3: ..G2, U$3.3
- removed net 4: ..+IN, U$3.4
- removed net 5: ..-VS, U$3.5
- removed net 6: ..REF, U$3.6
- removed net 7: ..VOUT, U$3.7
- removed net 8: ..+VS, U$3.8
- new net 3V3: C4.2, U$2.V2, U1.VOUT
- new net 5V: C3.2, U$2.V1, U1.ON/OFF, U1.VIN
- new net GND: C3.1, C4.1, U$2.GND@1, U$2.GND@2, U1.GND
Other:
- note added: "1.0"
- note removed: "1.0.0"
Changed lines of the file:
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@@
 <layer number="49" name="Reference" color="7" fill="1" visible="no" active="no"/>
 <layer number="50" name="dxf" color="7" fill="1" visible="no" active="no"/>
-<layer number="51" name="tDocu" color="14" fill="1" visible="no" active="no"/>
+<layer number="51" name="tDocu" color="7" fill="1" visible="no" active="no"/>
 <layer number="52" name="bDocu" color="7" fill="1" visible="no" active="no"/>
 <layer number="53" name="tGND_GNDA" color="7" fill="9" visible="no" active="no"/>
@@
 </classes>
 <parts>
-<part name="U$1" library="GClue" deviceset="A4L-LOC" device=""/>
-<part name="U$3" library="FaBo-Breakout" deviceset="8PIN" device=""/>
-<part name="." library="FaBo-Opamp" deviceset="ADA4075" device=""/>
+<part name="U$1" library="gclue" deviceset="A4L-LOC" device=""/>
+<part name="U1" library="FaBo-Supply" deviceset="LP2985" device="-33DBVR"/>
+<part name="SUPPLY5" library="FaBo-etc" deviceset="5V" device=""/>
+<part name="GND3" library="FaBo-etc" deviceset="GND" device=""/>
+<part name="C3" library="GClue-Capacitor" deviceset="CAPACITOR" device="0603" value="1uf"/>
+<part name="C4" library="GClue-Capacitor" deviceset="CAPACITOR" device="0603" value="1uf"/>
+<part name="GND4" library="FaBo-etc" deviceset="GND" device=""/>
+<part name="SUPPLY6" library="FaBo-etc" deviceset="3V3" device=""/>
+<part name="U$2" library="FaBo-Breakout" deviceset="4PIN-REGULATOR" device=""/>
+<part name="SUPPLY1" library="FaBo-etc" deviceset="5V" device=""/>
+<part name="SUPPLY2" library="FaBo-etc" deviceset="3V3" device=""/>
+<part name="GND1" library="FaBo-etc" deviceset="GND" device=""/>
 </parts>
 <sheets>
 <sheet>
 <plain>
-<text x="246.38" y="20.32" size="2.54" layer="94" align="bottom-center">1.0.0</text>
+<text x="246.38" y="20.32" size="2.54" layer="94" align="bottom-center">1.0</text>
 </plain>
 <instances>
 <instance part="U$1" gate="G$1" x="0" y="0"/>
-<instance part="U$3" gate="G$1" x="76.2" y="106.68"/>
-<instance part="." gate="G$1" x="76.2" y="137.16"/>
+<instance part="U1" gate="G$1" x="78.74" y="129.54"/>
+<instance part="SUPPLY5" gate="5V" x="33.02" y="142.24"/>
+<instance part="GND3" gate="GND" x="27.94" y="111.76"/>
+<instance part="C3" gate="G$1" x="33.02" y="127" rot="R90"/>
+<instance part="C4" gate="G$1" x="106.68" y="127" rot="R90"/>
+<instance part="GND4" gate="GND" x="106.68" y="119.38"/>
+<instance part="SUPPLY6" gate="3V3" x="106.68" y="144.78"/>
+<instance part="U$2" gate="G$1" x="160.02" y="129.54"/>
+<instance part="SUPPLY1" gate="5V" x="134.62" y="139.7"/>
+<instance part="SUPPLY2" gate="3V3" x="185.42" y="139.7"/>
+<instance part="GND1" gate="GND" x="162.56" y="104.14"/>
 </instances>
 <busses>
 </busses>
 <nets>
-<net name="1" class="0">
+<net name="GND" class="0">
 <segment>
-<wire x1="63.5" y1="139.7" x2="53.34" y2="139.7" width="0.1524" layer="91"/>
-<label x="53.34" y="139.7" size="1.778" layer="95"/>
-<pinref part="." gate="G$1" pin="-IN"/>
+<pinref part="U1" gate="G$1" pin="GND"/>
+<wire x1="63.5" y1="124.46" x2="33.02" y2="124.46" width="0.1524" layer="91"/>
+<wire x1="33.02" y1="124.46" x2="27.94" y2="124.46" width="0.1524" layer="91"/>
+<wire x1="27.94" y1="124.46" x2="27.94" y2="111.76" width="0.1524" layer="91"/>
+<pinref part="GND3" gate="GND" pin="GND"/>
+<pinref part="C3" gate="G$1" pin="1"/>
+<junction x="33.02" y="124.46"/>
 </segment>
 <segment>
-<wire x1="63.5" y1="109.22" x2="53.34" y2="109.22" width="0.1524" layer="91"/>
-<label x="53.34" y="109.22" size="1.778" layer="95"/>
-<pinref part="U$3" gate="G$1" pin="1"/>
+<pinref part="GND4" gate="GND" pin="GND"/>
+<pinref part="C4" gate="G$1" pin="1"/>
+<wire x1="106.68" y1="119.38" x2="106.68" y2="124.46" width="0.1524" layer="91"/>
+</segment>
+<segment>
+<pinref part="U$2" gate="G$1" pin="GND@1"/>
+<wire x1="149.86" y1="127" x2="134.62" y2="127" width="0.1524" layer="91"/>
+<wire x1="134.62" y1="127" x2="134.62" y2="116.84" width="0.1524" layer="91"/>
+<wire x1="134.62" y1="116.84" x2="162.56" y2="116.84" width="0.1524" layer="91"/>
+<wire x1="162.56" y1="116.84" x2="185.42" y2="116.84" width="0.1524" layer="91"/>
+<wire x1="185.42" y1="116.84" x2="185.42" y2="127" width="0.1524" layer="91"/>
+<pinref part="U$2" gate="G$1" pin="GND@2"/>
+<wire x1="185.42" y1="127" x2="172.72" y2="127" width="0.1524" layer="91"/>
+<wire x1="162.56" y1="116.84" x2="162.56" y2="104.14" width="0.1524" layer="91"/>
+<pinref part="GND1" gate="GND" pin="GND"/>
 </segment>
 </net>
-<net name="2" class="0">
+<net name="3V3" class="0">
 <segment>
-<wire x1="63.5" y1="137.16" x2="53.34" y2="137.16" width="0.1524" layer="91"/>
-<label x="53.34" y="137.16" size="1.778" layer="95"/>
-<pinref part="." gate="G$1" pin="G1"/>
+<pinref part="U1" gate="G$1" pin="VOUT"/>
+<wire x1="93.98" y1="134.62" x2="106.68" y2="134.62" width="0.1524" layer="91"/>
+<wire x1="106.68" y1="134.62" x2="106.68" y2="144.78" width="0.1524" layer="91"/>
+<pinref part="C4" gate="G$1" pin="2"/>
+<wire x1="106.68" y1="132.08" x2="106.68" y2="134.62" width="0.1524" layer="91"/>
+<pinref part="SUPPLY6" gate="3V3" pin="3V3"/>
 </segment>
 <segment>
-<wire x1="63.5" y1="106.68" x2="53.34" y2="106.68" width="0.1524" layer="91"/>
-<label x="53.34" y="106.68" size="1.778" layer="95"/>
-<pinref part="U$3" gate="G$1" pin="2"/>
+<pinref part="U$2" gate="G$1" pin="V2"/>
+<wire x1="172.72" y1="132.08" x2="185.42" y2="132.08" width="0.1524" layer="91"/>
+<wire x1="185.42" y1="132.08" x2="185.42" y2="139.7" width="0.1524" layer="91"/>
+<pinref part="SUPPLY2" gate="3V3" pin="3V3"/>
 </segment>
 </net>
-<net name="3" class="0">
+<net name="5V" class="0">
 <segment>
-<wire x1="63.5" y1="134.62" x2="53.34" y2="134.62" width="0.1524" layer="91"/>
-<label x="53.34" y="134.62" size="1.778" layer="95"/>
-<pinref part="." gate="G$1" pin="G2"/>
+<pinref part="SUPPLY5" gate="5V" pin="5V"/>
+<pinref part="U1" gate="G$1" pin="VIN"/>
+<wire x1="33.02" y1="142.24" x2="33.02" y2="134.62" width="0.1524" layer="91"/>
+<wire x1="33.02" y1="134.62" x2="50.8" y2="134.62" width="0.1524" layer="91"/>
+<wire x1="50.8" y1="134.62" x2="63.5" y2="134.62" width="0.1524" layer="91"/>
+<wire x1="50.8" y1="134.62" x2="50.8" y2="129.54" width="0.1524" layer="91"/>
+<pinref part="U1" gate="G$1" pin="ON/OFF"/>
+<wire x1="50.8" y1="129.54" x2="63.5" y2="129.54" width="0.1524" layer="91"/>
+<pinref part="C3" gate="G$1" pin="2"/>
+<wire x1="33.02" y1="132.08" x2="33.02" y2="134.62" width="0.1524" layer="91"/>
 </segment>
 <segment>
-<wire x1="63.5" y1="104.14" x2="53.34" y2="104.14" width="0.1524" layer="91"/>
-<label x="53.34" y="104.14" size="1.778" layer="95"/>
-<pinref part="U$3" gate="G$1" pin="3"/>
+<pinref part="U$2" gate="G$1" pin="V1"/>
+<wire x1="149.86" y1="132.08" x2="134.62" y2="132.08" width="0.1524" layer="91"/>
+<wire x1="134.62" y1="132.08" x2="134.62" y2="139.7" width="0.1524" layer="91"/>
+<pinref part="SUPPLY1" gate="5V" pin="5V"/>
 </segment>
 </net>
-<net name="4" class="0">
-<segment>
-<wire x1="63.5" y1="132.08" x2="53.34" y2="132.08" width="0.1524" layer="91"/>
-<label x="53.34" y="132.08" size="1.778" layer="95"/>
-<pinref part="." gate="G$1" pin="+IN"/>
-</segment>
-<segment>
-<wire x1="63.5" y1="101.6" x2="53.34" y2="101.6" width="0.1524" layer="91"/>
-<label x="53.34" y="101.6" size="1.778" layer="95"/>
-<pinref part="U$3" gate="G$1" pin="4"/>
-</segment>
-</net>
-<net name="8" class="0">
-<segment>
-<wire x1="88.9" y1="109.22" x2="101.6" y2="109.22" width="0.1524" layer="91"/>
-<label x="101.6" y="109.22" size="1.778" layer="95"/>
-<pinref part="U$3" gate="G$1" pin="8"/>
-</segment>
-<segment>
-<wire x1="88.9" y1="139.7" x2="99.06" y2="139.7" width="0.1524" layer="91"/>
-<label x="99.06" y="139.7" size="1.778" layer="95"/>
-<pinref part="." gate="G$1" pin="+VS"/>
-</segment>
-</net>
-<net name="7" class="0">
-<segment>
-<wire x1="88.9" y1="106.68" x2="101.6" y2="106.68" width="0.1524" layer="91"/>
-<label x="101.6" y="106.68" size="1.778" layer="95"/>
-<pinref part="U$3" gate="G$1" pin="7"/>
-</segment>
-<segment>
-<wire x1="88.9" y1="137.16" x2="99.06" y2="137.16" width="0.1524" layer="91"/>
-<label x="99.06" y="137.16" size="1.778" layer="95"/>
-<pinref part="." gate="G$1" pin="VOUT"/>
-</segment>
-</net>
-<net name="6" class="0">
-<segment>
-<wire x1="88.9" y1="104.14" x2="101.6" y2="104.14" width="0.1524" layer="91"/>
-<label x="101.6" y="104.14" size="1.778" layer="95"/>
-<pinref part="U$3" gate="G$1" pin="6"/>
-</segment>
-<segment>
-<wire x1="88.9" y1="134.62" x2="99.06" y2="134.62" width="0.1524" layer="91"/>
-<label x="99.06" y="134.62" size="1.778" layer="95"/>
-<pinref part="." gate="G$1" pin="REF"/>
-</segment>
-</net>
-<net name="5" class="0">
-<segment>
-<wire x1="88.9" y1="101.6" x2="101.6" y2="101.6" width="0.1524" layer="91"/>
-<label x="101.6" y="101.6" size="1.778" layer="95"/>
-<pinref part="U$3" gate="G$1" pin="5"/>
-</segment>
-<segment>
-<wire x1="88.9" y1="132.08" x2="99.06" y2="132.08" width="0.1524" layer="91"/>
-<label x="99.06" y="132.08" size="1.778" layer="95"/>
-<pinref part="." gate="G$1" pin="-VS"/>
-</segment>
-</net>
