File: MPL3115/MPL3115_breakout.sch (EAGLE design)
At the start: 2 parts

Commit message: Update new meme.
Parts:
- removed .: ADA4075, FaBo-Opamp:ADA4075
- removed U$3: 8PIN, FaBo-Breakout:8PIN
- added MPL3115A1: FS-MPL3115A2, FaBo-Mems:FS-MPL3115A2
- added U$1: 8PIN, FaBo-Breakout:8PIN
Connections:
- removed net 1: ..-IN, U$3.1
- removed net 2: ..G1, U$3.2
- removed net 3: ..G2, U$3.3
- removed net 4: ..+IN, U$3.4
- removed net 5: ..-VS, U$3.5
- removed net 6: ..REF, U$3.6
- removed net 7: ..VOUT, U$3.7
- removed net 8: ..+VS, U$3.8
- new net CAP: MPL3115A1.CAP, U$1.2
- new net GND: MPL3115A1.GND, U$1.3
- new net INT1: MPL3115A1.INT1, U$1.6
- new net INT2: MPL3115A1.INT2, U$1.5
- new net SCL: MPL3115A1.SCL, U$1.8
- new net SDA: MPL3115A1.SDA, U$1.7
- new net VDD: MPL3115A1.VDD, U$1.1
- new net VDDIO: MPL3115A1.VDDIO, U$1.4
Other:
- note removed: "1.0.0"
Changed lines of the file:
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@@
 <layer number="49" name="Reference" color="7" fill="1" visible="no" active="no"/>
 <layer number="50" name="dxf" color="7" fill="1" visible="no" active="no"/>
-<layer number="51" name="tDocu" color="14" fill="1" visible="no" active="no"/>
+<layer number="51" name="tDocu" color="7" fill="1" visible="no" active="no"/>
 <layer number="52" name="bDocu" color="7" fill="1" visible="no" active="no"/>
 <layer number="53" name="tGND_GNDA" color="7" fill="9" visible="no" active="no"/>
@@
 <layer number="154" name="FabDoc2" color="2" fill="1" visible="no" active="no"/>
 <layer number="155" name="FabDoc3" color="7" fill="15" visible="no" active="no"/>
-<layer number="160" name="O_Dim" color="12" fill="11" visible="yes" active="yes"/>
 <layer number="199" name="Contour" color="7" fill="1" visible="yes" active="yes"/>
-<layer number="200" name="200bmp" color="1" fill="10" visible="yes" active="yes"/>
+<layer number="200" name="200bmp" color="1" fill="10" visible="no" active="yes"/>
 <layer number="201" name="201bmp" color="2" fill="1" visible="no" active="no"/>
 <layer number="202" name="202bmp" color="3" fill="1" visible="no" active="no"/>
@@
 </classes>
 <parts>
-<part name="U$1" library="GClue" deviceset="A4L-LOC" device=""/>
-<part name="U$3" library="FaBo-Breakout" deviceset="8PIN" device=""/>
-<part name="." library="FaBo-Opamp" deviceset="ADA4075" device=""/>
+<part name="U$1" library="FaBo-Breakout" deviceset="8PIN" device=""/>
+<part name="MPL3115A1" library="FaBo-Mems" deviceset="FS-MPL3115A2" device=""/>
 </parts>
 <sheets>
 <sheet>
 <plain>
-<text x="246.38" y="20.32" size="2.54" layer="94" align="bottom-center">1.0.0</text>
 </plain>
 <instances>
-<instance part="U$1" gate="G$1" x="0" y="0"/>
-<instance part="U$3" gate="G$1" x="76.2" y="106.68"/>
-<instance part="." gate="G$1" x="76.2" y="137.16"/>
+<instance part="U$1" gate="G$1" x="43.18" y="63.5"/>
+<instance part="MPL3115A1" gate="G$1" x="43.18" y="33.02"/>
 </instances>
 <busses>
 </busses>
 <nets>
-<net name="1" class="0">
-<segment>
-<wire x1="63.5" y1="139.7" x2="53.34" y2="139.7" width="0.1524" layer="91"/>
-<label x="53.34" y="139.7" size="1.778" layer="95"/>
-<pinref part="." gate="G$1" pin="-IN"/>
-</segment>
-<segment>
-<wire x1="63.5" y1="109.22" x2="53.34" y2="109.22" width="0.1524" layer="91"/>
-<label x="53.34" y="109.22" size="1.778" layer="95"/>
-<pinref part="U$3" gate="G$1" pin="1"/>
-</segment>
-</net>
-<net name="2" class="0">
-<segment>
-<wire x1="63.5" y1="137.16" x2="53.34" y2="137.16" width="0.1524" layer="91"/>
-<label x="53.34" y="137.16" size="1.778" layer="95"/>
-<pinref part="." gate="G$1" pin="G1"/>
-</segment>
-<segment>
-<wire x1="63.5" y1="106.68" x2="53.34" y2="106.68" width="0.1524" layer="91"/>
-<label x="53.34" y="106.68" size="1.778" layer="95"/>
-<pinref part="U$3" gate="G$1" pin="2"/>
-</segment>
-</net>
-<net name="3" class="0">
-<segment>
-<wire x1="63.5" y1="134.62" x2="53.34" y2="134.62" width="0.1524" layer="91"/>
-<label x="53.34" y="134.62" size="1.778" layer="95"/>
-<pinref part="." gate="G$1" pin="G2"/>
-</segment>
-<segment>
-<wire x1="63.5" y1="104.14" x2="53.34" y2="104.14" width="0.1524" layer="91"/>
-<label x="53.34" y="104.14" size="1.778" layer="95"/>
-<pinref part="U$3" gate="G$1" pin="3"/>
-</segment>
-</net>
-<net name="4" class="0">
-<segment>
-<wire x1="63.5" y1="132.08" x2="53.34" y2="132.08" width="0.1524" layer="91"/>
-<label x="53.34" y="132.08" size="1.778" layer="95"/>
-<pinref part="." gate="G$1" pin="+IN"/>
-</segment>
-<segment>
-<wire x1="63.5" y1="101.6" x2="53.34" y2="101.6" width="0.1524" layer="91"/>
-<label x="53.34" y="101.6" size="1.778" layer="95"/>
-<pinref part="U$3" gate="G$1" pin="4"/>
-</segment>
-</net>
-<net name="8" class="0">
-<segment>
-<wire x1="88.9" y1="109.22" x2="101.6" y2="109.22" width="0.1524" layer="91"/>
-<label x="101.6" y="109.22" size="1.778" layer="95"/>
-<pinref part="U$3" gate="G$1" pin="8"/>
-</segment>
-<segment>
-<wire x1="88.9" y1="139.7" x2="99.06" y2="139.7" width="0.1524" layer="91"/>
-<label x="99.06" y="139.7" size="1.778" layer="95"/>
-<pinref part="." gate="G$1" pin="+VS"/>
-</segment>
-</net>
-<net name="7" class="0">
-<segment>
-<wire x1="88.9" y1="106.68" x2="101.6" y2="106.68" width="0.1524" layer="91"/>
-<label x="101.6" y="106.68" size="1.778" layer="95"/>
-<pinref part="U$3" gate="G$1" pin="7"/>
-</segment>
-<segment>
-<wire x1="88.9" y1="137.16" x2="99.06" y2="137.16" width="0.1524" layer="91"/>
-<label x="99.06" y="137.16" size="1.778" layer="95"/>
-<pinref part="." gate="G$1" pin="VOUT"/>
-</segment>
-</net>
-<net name="6" class="0">
-<segment>
-<wire x1="88.9" y1="104.14" x2="101.6" y2="104.14" width="0.1524" layer="91"/>
-<label x="101.6" y="104.14" size="1.778" layer="95"/>
-<pinref part="U$3" gate="G$1" pin="6"/>
-</segment>
-<segment>
-<wire x1="88.9" y1="134.62" x2="99.06" y2="134.62" width="0.1524" layer="91"/>
-<label x="99.06" y="134.62" size="1.778" layer="95"/>
-<pinref part="." gate="G$1" pin="REF"/>
-</segment>
-</net>
-<net name="5" class="0">
-<segment>
-<wire x1="88.9" y1="101.6" x2="101.6" y2="101.6" width="0.1524" layer="91"/>
-<label x="101.6" y="101.6" size="1.778" layer="95"/>
-<pinref part="U$3" gate="G$1" pin="5"/>
-</segment>
-<segment>
-<wire x1="88.9" y1="132.08" x2="99.06" y2="132.08" width="0.1524" layer="91"/>
-<label x="99.06" y="132.08" size="1.778" layer="95"/>
-<pinref part="." gate="G$1" pin="-VS"/>
-</segment>
-</net>
+<net name="VDD" class="0">
+<segment>
+<pinref part="U$1" gate="G$1" pin="1"/>
+<wire x1="30.48" y1="66.04" x2="15.24" y2="66.04" width="0.1524" layer="91"/>
+<label x="15.24" y="66.04" size="1.778" layer="95"/>
+</segment>
+<segment>
+<pinref part="MPL3115A1" gate="G$1" pin="VDD"/>
+<wire x1="30.48" y1="38.1" x2="17.78" y2="38.1" width="0.1524" layer="91"/>
+<label x="17.78" y="38.1" size="1.778" layer="95"/>
+</segment>
+</net>
+<net name="CAP" class="0">
+<segment>
+<pinref part="U$1" gate="G$1" pin="2"/>
+<wire x1="30.48" y1="63.5" x2="15.24" y2="63.5" width="0.1524" layer="91"/>
+<label x="15.24" y="63.5" size="1.778" layer="95"/>
+</segment>
+<segment>
+<pinref part="MPL3115A1" gate="G$1" pin="CAP"/>
+<wire x1="30.48" y1="35.56" x2="17.78" y2="35.56" width="0.1524" layer="91"/>
+<label x="17.78" y="35.56" size="1.778" layer="95"/>
+</segment>
+</net>
+<net name="GND" class="0">
+<segment>
+<pinref part="U$1" gate="G$1" pin="3"/>
+<wire x1="30.48" y1="60.96" x2="15.24" y2="60.96" width="0.1524" layer="91"/>
+<label x="15.24" y="60.96" size="1.778" layer="95"/>
+</segment>
+<segment>
+<pinref part="MPL3115A1" gate="G$1" pin="GND"/>
+<wire x1="30.48" y1="33.02" x2="17.78" y2="33.02" width="0.1524" layer="91"/>
+<label x="17.78" y="33.02" size="1.778" layer="95"/>
+</segment>
+</net>
+<net name="VDDIO" class="0">
+<segment>
+<pinref part="U$1" gate="G$1" pin="4"/>
+<wire x1="30.48" y1="58.42" x2="15.24" y2="58.42" width="0.1524" layer="91"/>
+<label x="15.24" y="58.42" size="1.778" layer="95"/>
+</segment>
+<segment>
+<pinref part="MPL3115A1" gate="G$1" pin="VDDIO"/>
+<wire x1="30.48" y1="30.48" x2="17.78" y2="30.48" width="0.1524" layer="91"/>
+<label x="17.78" y="30.48" size="1.778" layer="95"/>
+</segment>
+</net>
+<net name="SCL" class="0">
+<segment>
+<pinref part="U$1" gate="G$1" pin="8"/>
+<wire x1="55.88" y1="66.04" x2="71.12" y2="66.04" width="0.1524" layer="91"/>
+<label x="71.12" y="66.04" size="1.778" layer="95"/>
+</segment>
+<segment>
+<pinref part="MPL3115A1" gate="G$1" pin="SCL"/>
+<wire x1="55.88" y1="38.1" x2="68.58" y2="38.1" width="0.1524" layer="91"/>
+<label x="68.58" y="38.1" size="1.778" layer="95"/>
+</segment>
+</net>
+<net name="SDA" class="0">
+<segment>
+<pinref part="U$1" gate="G$1" pin="7"/>
+<wire x1="55.88" y1="63.5" x2="71.12" y2="63.5" width="0.1524" layer="91"/>
+<label x="71.12" y="63.5" size="1.778" layer="95"/>
+</segment>
+<segment>
+<pinref part="MPL3115A1" gate="G$1" pin="SDA"/>
+<wire x1="55.88" y1="35.56" x2="68.58" y2="35.56" width="0.1524" layer="91"/>
+<label x="68.58" y="35.56" size="1.778" layer="95"/>
+</segment>
+</net>
+<net name="INT1" class="0">
+<segment>
+<pinref part="U$1" gate="G$1" pin="6"/>
+<wire x1="55.88" y1="60.96" x2="71.12" y2="60.96" width="0.1524" layer="91"/>
+<label x="71.12" y="60.96" size="1.778" layer="95"/>
+</segment>
+<segment>
+<pinref part="MPL3115A1" gate="G$1" pin="INT1"/>
+<wire x1="55.88" y1="33.02" x2="68.58" y2="33.02" width="0.1524" layer="91"/>
+<label x="68.58" y="33.02" size="1.778" layer="95"/>
+</segment>
+</net>
+<net name="INT2" class="0">
+<segment>
+<pinref part="U$1" gate="G$1" pin="5"/>
+<wire x1="55.88" y1="58.42" x2="71.12" y2="58.42" width="0.1524" layer="91"/>
+<label x="71.12" y="58.42" size="1.778" layer="95"/>
+</segment>
+<segment>
+<wire x1="68.58" y1="30.48" x2="55.88" y2="30.48" width="0.1524" layer="91"/>
+<pinref part="MPL3115A1" gate="G$1" pin="INT2"/>
+<label x="68.58" y="30.48" size="1.778" layer="95"/>
+</segment>
+</net>
