File: VNC2/VNC2.brd (EAGLE design)
At the start: 21.6 x 39.4 mm, 23 parts, among them Q1 12MHz

Commit message: fix dimension
Parts:
- C10, C11: value 0.1uF -> 1uF
Other:
- outline, holes or cut-outs redrawn
Changed lines of the file:
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@@
 <board>
 <plain>
-<wire x1="0" y1="0" x2="21.59" y2="0" width="0" layer="20"/>
-<wire x1="21.59" y1="0" x2="21.59" y2="39.37" width="0" layer="20"/>
-<wire x1="21.59" y1="39.37" x2="0" y2="39.37" width="0" layer="20"/>
-<wire x1="0" y1="39.37" x2="0" y2="0" width="0" layer="20"/>
+<wire x1="21.59" y1="1.27" x2="21.59" y2="38.1" width="0" layer="20"/>
+<wire x1="0" y1="38.1" x2="0" y2="1.27" width="0" layer="20"/>
 <text x="10.795" y="3.556" size="0.8128" layer="21" font="vector" ratio="12" align="bottom-center">DEBUG</text>
-<dimension x1="26.035" y1="0" x2="26.035" y2="39.37" x3="31.115" y3="19.685" textsize="1.778" layer="51" visible="yes"/>
+<dimension x1="22.86" y1="0" x2="22.86" y2="39.37" x3="27.94" y3="19.685" textsize="1.778" layer="51" visible="yes"/>
 <text x="4.445" y="3.556" size="0.8128" layer="22" font="vector" ratio="12" rot="MR90" align="center-left">DBG</text>
 <text x="3.556" y="22.86" size="0.8128" layer="21" font="vector" ratio="12" align="center-left">5V</text>
@@
 <text x="14.605" y="3.556" size="0.8128" layer="22" font="vector" ratio="12" rot="MR90" align="center-left">PRG</text>
 <text x="17.145" y="3.556" size="0.8128" layer="22" font="vector" ratio="12" rot="MR90" align="center-left">VCC</text>
+<dimension x1="0" y1="-1.27" x2="21.59" y2="-1.27" x3="10.795" y3="-5.715" textsize="1.778" layer="51" visible="yes"/>
+<wire x1="1.27" y1="0" x2="20.32" y2="0" width="0" layer="20"/>
+<wire x1="1.27" y1="39.37" x2="20.32" y2="39.37" width="0" layer="20"/>
+<wire x1="0" y1="38.1" x2="1.27" y2="39.37" width="0" layer="20" curve="-90"/>
+<wire x1="1.27" y1="0" x2="0" y2="1.27" width="0" layer="20" curve="-90"/>
+<wire x1="21.59" y1="1.27" x2="20.32" y2="0" width="0" layer="20" curve="-90"/>
+<wire x1="20.32" y1="39.37" x2="21.59" y2="38.1" width="0" layer="20" curve="-90"/>
 </plain>
 <attributes>
@@
 <attribute name="VALUE" x="6.35" y="29.21" size="0.8128" layer="27" font="vector" ratio="12" align="center"/>
 </element>
-<element name="C10" library="FaBo-Capacitor" package="0603-NARROW" value="0.1uF" x="6.223" y="26.162" smashed="yes" rot="R90">
+<element name="C10" library="FaBo-Capacitor" package="0603-NARROW" value="1uF" x="6.223" y="26.162" smashed="yes" rot="R90">
 <attribute name="NAME" x="5.461" y="26.162" size="0.6096" layer="25" font="vector" ratio="12" rot="R90" align="bottom-center"/>
 <attribute name="VALUE" x="6.223" y="26.162" size="0.8128" layer="27" font="vector" ratio="12" rot="R90" align="center"/>
 </element>
-<element name="C11" library="FaBo-Capacitor" package="0603-NARROW" value="0.1uF" x="13.97" y="26.162" smashed="yes" rot="R90">
+<element name="C11" library="FaBo-Capacitor" package="0603-NARROW" value="1uF" x="13.97" y="26.162" smashed="yes" rot="R90">
 <attribute name="NAME" x="14.732" y="26.162" size="0.6096" layer="25" font="vector" ratio="12" rot="R270" align="bottom-center"/>
 <attribute name="VALUE" x="13.97" y="26.162" size="0.8128" layer="27" font="vector" ratio="12" rot="R90" align="center"/>
