File: BT121/BT121breakout.brd (EAGLE design)
At the start: 34.3 x 34.3 mm, 4 parts

Commit message: change bt121
Parts:
- moved CN2 16.5 mm to (48.9, 17.1)
- moved U1 8.36 mm to (25.5, 27.3)
- moved CN3 8.25 mm to (25.4, 1.91)
Routing:
- net PA6: track 13.1 -> 21.4 mm
- net PA7: track 12.4 -> 20.8 mm
- net VDD: track 12.4 -> 20.6 mm
- net PA5: track 14.3 -> 22.1 mm
- net PA10: track 14.3 -> 21.9 mm
- net PA9: track 13.9 -> 21.2 mm
- net PA4: track 15.9 -> 22.7 mm
- net PB3: track 17.3 -> 23.3 mm
- net PB4: track 18.1 -> 24.0 mm
- net PA12: track 17.4 -> 23.1 mm
- net PA14: track 18.2 -> 23.8 mm
- net PA11: track 17.0 -> 22.5 mm
- net RESET: track 23.5 -> 26.4 mm
- net PB7: track 23.5 -> 26.3 mm
- net PB6: track 23.0 -> 25.3 mm
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Other:
- board size 34.3 x 34.3 mm -> 51 x 34.3 mm
- board text added: "-20-"
- board text added: "Rev. BETA2"
- board text removed: "Rev. BETA"
