File: BT121/BT121breakout.sch (EAGLE design)
At the start: 4 parts

Commit message: change bt121
Other:
- note added: "Beta2"
- note removed: "Beta"
Changed lines of the file:
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@@
 <setting verticaltext="up"/>
 </settings>
-<grid distance="0.1" unitdist="inch" unit="inch" style="lines" multiple="1" display="yes" altdistance="0.01" altunitdist="inch" altunit="inch"/>
+<grid distance="0.1" unitdist="inch" unit="inch" style="lines" multiple="1" display="no" altdistance="0.01" altunitdist="inch" altunit="inch"/>
 <layers>
 <layer number="1" name="Top" color="4" fill="1" visible="no" active="no"/>
@@
 <sheet>
 <plain>
-<text x="246.38" y="20.32" size="2.54" layer="94" align="bottom-center">Beta</text>
+<text x="246.38" y="20.32" size="2.54" layer="94" align="bottom-center">Beta2</text>
 </plain>
 <instances>
